File: FrameworkThinkpadSharedSplit.kicad_pcb (KiCad board)
At the start: 2 copper layers, 148 parts, among them J1 Conn_01x05_Socket, J10 Conn_01x03_Socket, J11 Conn_01x06_Socket, J2 Conn_01x05_Socket, J3 Conn_01x05_Socket, J4 Conn_01x07_Socket, J5 Conn_01x07_Socket, J6 Conn_01x07_Socket, J7 Conn_01x07_Socket, J8 Conn_01x05_Socket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

Commit message: added wiring to most parts
Parts:
- removed J9: Conn_01x03_Socket, Connector_Molex:Molex_PicoBlade_53048-0310_1x03_P1.25mm_Horizontal
- added D29: LED, LED_THT:LED_D5.0mm, F.Cu at (279.5, 28.5)
- added D31: LED, LED_THT:LED_D5.0mm, F.Cu at (296.5, 28.5)
- added D32: LED, LED_THT:LED_D5.0mm, F.Cu at (305.0, 28.5)
- added J12: Conn_01x06_Socket, Connector_Molex:Molex_PicoBlade_53048-0610_1x06_P1.25mm_Horizontal, F.Cu at (263.4, 32.8)
- added R1: Resistor 82Ω, Resistor_THT:R_Axial_DIN0207_L6.3mm_D2.5mm_P7.62mm_Horizontal, F.Cu at (282.5, 32.5)
- added R2: Resistor 82Ω, Resistor_THT:R_Axial_DIN0207_L6.3mm_D2.5mm_P7.62mm_Horizontal, F.Cu at (291.0, 36.0)
- added R3: Resistor 82Ω, Resistor_THT:R_Axial_DIN0207_L6.3mm_D2.5mm_P7.62mm_Horizontal, F.Cu at (298.8, 32.5)
- added R4: Resistor 82Ω, Resistor_THT:R_Axial_DIN0207_L6.3mm_D2.5mm_P7.62mm_Horizontal, F.Cu at (306.5, 36.0)
- added R5: Resistor 82Ω, Resistor_THT:R_Axial_DIN0207_L6.3mm_D2.5mm_P7.62mm_Horizontal, F.Cu at (315.5, 33.0)
- added REF**: MountingHole_4.5mm, MountingHole:MountingHole_4.5mm, F.Cu at (36.0, 130.0)
- added REF**: MountingHole_4.5mm, MountingHole:MountingHole_4.5mm, F.Cu at (322.5, 33.0)
- added REF**: MountingHole_4.5mm, MountingHole:MountingHole_4.5mm, F.Cu at (141.0, 205.0)
- added REF**: MountingHole_4.5mm, MountingHole:MountingHole_4.5mm, F.Cu at (182.5, 140.0)
- added REF**: MountingHole_4.5mm, MountingHole:MountingHole_4.5mm, F.Cu at (30.5, 56.0)
- added REF**: MountingHole_4.5mm, MountingHole:MountingHole_4.5mm, F.Cu at (249.5, 33.0)
- added REF**: MountingHole_4.5mm, MountingHole:MountingHole_4.5mm, F.Cu at (170.5, 140.0)
- added REF**: MountingHole_4.5mm, MountingHole:MountingHole_4.5mm, F.Cu at (169.5, 55.0)
- added REF**: MountingHole_4.5mm, MountingHole:MountingHole_4.5mm, F.Cu at (36.0, 204.0)
- added REF**: MountingHole_4.5mm, MountingHole:MountingHole_4.5mm, F.Cu at (183.5, 55.0)
- added REF**: MountingHole_4.5mm, MountingHole:MountingHole_4.5mm, F.Cu at (36.0, 163.0)
- added REF**: MountingHole_4.5mm, MountingHole:MountingHole_4.5mm, F.Cu at (322.5, 57.0)
- added REF**: MountingHole_4.5mm, MountingHole:MountingHole_4.5mm, F.Cu at (141.0, 163.0)
- added REF**: MountingHole_4.5mm, MountingHole:MountingHole_4.5mm, F.Cu at (317.0, 130.0)
- added U2: Arduino_Pro_Micro, ScottoKeebs_MCU:Arduino_Pro_Micro, F.Cu at (126.0, 189.5)
- J10: value Conn_01x03_Socket -> Conn_01x06_Socket; footprint Connector_Molex:Molex_PicoBlade_53048-0310_1x03_P1.25mm_Horizontal -> Connector_Molex:Molex_PicoBlade_53048-0610_1x06_P1.25mm_Horizontal
- moved J10 215.5 mm to (114.0, 174.0), turned to 180 degrees
- moved TP1 81.1 mm to (43.0, 171.0)
- moved TP10 81.1 mm to (46.5, 162.0)
- moved TP2 81.1 mm to (44.4, 171.0)
- moved TP3 81.1 mm to (45.9, 171.0)
- moved TP4 81.1 mm to (48.0, 171.0)
- moved TP5 81.1 mm to (54.0, 162.0)
- moved TP6 81.1 mm to (52.5, 161.0)
- moved TP7 81.1 mm to (51.0, 161.0)
- moved TP8 81.1 mm to (49.5, 161.0)
- moved TP9 81.1 mm to (48.0, 161.0)
- moved J11 80.1 mm to (96.9, 169.0), turned to 0 degrees
- moved J6 66.5 mm to (94.0, 203.0), turned to 0 degrees
- moved U1 45.8 mm to (76.9, 189.2)
- moved J5 40.4 mm to (196.2, 49.7)
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- renumbered D29 to D67
Connections:
- D67 pad 1: Net-(D29-K) -> Net-(D67-K)
- J10 pad 1: Net-(D29-A) -> Power LED GND
- J10 pad 2: Net-(D29-K) -> Numpad Led
- J10 pad 3: Net-(D30-K) -> Caps Led
- S33 pad 1: unconnected-(S33-Pad1) -> Net-(J7-Pin_5)
- TP4 pad 1: LED PWR -> Trackpoint PWR
- U1 pad 27: LED PWR -> Trackpoint PWR
- U1 pad 30: unconnected-(U1-5v-Pad30) -> LED PWR
- U1 pad 4: unconnected-(U1-GND-Pad4) -> Power LED GND
Routing:
- net Net-(D33-K): track 0.00 -> 233.7 mm
- net Net-(D22-K): track 0.00 -> 221.4 mm
- net Net-(D15-K): track 0.00 -> 197.4 mm
- net Net-(D57-K): track 0.00 -> 187.5 mm
- net Net-(J7-Pin_7): track 0.00 -> 181.3 mm
- net Net-(D50-K): track 0.00 -> 170.0 mm
- net Net-(J5-Pin_7): track 0.00 -> 167.4 mm
- net Net-(D1-K): track 0.00 -> 165.6 mm
- net Net-(D10-K): track 0.00 -> 164.0 mm
- net Net-(J7-Pin_6): track 0.00 -> 163.9 mm
- net Net-(D36-K): track 0.00 -> 159.8 mm
- net Net-(D43-K): track 0.00 -> 159.2 mm
- net Net-(J5-Pin_6): track 0.00 -> 150.1 mm
- net Net-(J7-Pin_5): track 0.00 -> 146.6 mm
- net Net-(J5-Pin_5): track 0.00 -> 133.2 mm
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
Commit message: moved pcbs around
Parts:
- moved REF** 133.3 mm to (137.1, 71.8)
- moved REF** 133.3 mm to (32.1, 70.8)
- moved REF** 133.3 mm to (32.1, 29.8)
- moved REF** 133.3 mm to (137.1, 29.8)
- moved TP1 133.3 mm to (39.1, 37.8)
- moved TP10 133.3 mm to (42.6, 28.8)
- moved TP2 133.3 mm to (40.5, 37.8)
- moved TP3 133.3 mm to (42.0, 37.8)
- moved TP4 133.3 mm to (44.1, 37.8)
- moved TP5 133.3 mm to (50.1, 28.8)
- moved TP6 133.3 mm to (48.6, 27.8)
- moved TP7 133.3 mm to (47.1, 27.8)
- moved TP8 133.3 mm to (45.6, 27.8)
- moved TP9 133.3 mm to (44.1, 27.8)
- moved J10 130.6 mm to (110.0, 43.4)
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Routing:
- net Net-(J7-Pin_4): track 109.4 -> 114.4 mm
- net Net-(J7-Pin_6): track 163.9 -> 168.9 mm
- net Net-(J7-Pin_5): track 146.6 -> 151.5 mm
- net Net-(J7-Pin_7): track 181.3 -> 186.2 mm
- net Net-(J7-Pin_3): track 95.1 -> 99.5 mm
- net Net-(J7-Pin_2): track 77.9 -> 81.7 mm
- net Net-(J7-Pin_1): track 68.2 -> 65.4 mm
- net Net-(J12-Pin_4): track 29.8 -> 30.0 mm, vias 1 -> 3
- net Net-(J12-Pin_2): vias 3 -> 1
Other:
- board outline added: 297.2 x 158.5 mm

Commit message: changed how board is connected to handle paneling
Parts:
- moved D16 12.4 mm to (69.8, 144.5)
- moved D18 12.4 mm to (107.8, 144.5)
- moved D24 12.4 mm to (88.8, 162.5)
- moved D25 12.4 mm to (106.8, 162.5)
- moved D27 12.4 mm to (144.8, 161.5)
- moved D33 12.4 mm to (125.8, 179.5)
- moved D35 12.4 mm to (162.8, 179.5)
- moved D22 12.4 mm to (51.8, 161.5)
- moved REF** 12.4 mm to (33.8, 180.5)
- moved D10 12.4 mm to (88.8, 127.2)
- moved D11 12.4 mm to (106.8, 127.2)
- moved D12 12.4 mm to (125.8, 127.2)
- moved D3 12.4 mm to (88.8, 109.2)
- moved D4 12.4 mm to (106.8, 109.2)
- moved D6 12.4 mm to (144.8, 109.2)
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Other:
- board size 297.2 x 158.5 mm -> 298.1 x 158.9 mm
