File: FrameworkThinkpadSharedSplit.kicad_sch (KiCad schematic)
At the start: 148 parts, among them J1 Conn_01x05_Socket, J10 Conn_01x03_Socket, J11 Conn_01x06_Socket, J2 Conn_01x05_Socket, J3 Conn_01x05_Socket, J4 Conn_01x07_Socket, J5 Conn_01x07_Socket, J6 Conn_01x07_Socket, J7 Conn_01x07_Socket, J8 Conn_01x05_Socket, J9 Conn_01x03_Socket, U1 RP2040_Pro_Micro

Commit message: added wiring to most parts
Parts:
- removed J10, J9: Conn_01x03_Socket, Connector_Molex:Molex_PicoBlade_53048-0310_1x03_P1.25mm_Horizontal, symbol Connector:Conn_01x03_Socket
- added D31, D32, D67: LED, LED_THT:LED_D5.0mm, symbol Device:LED
- added J10, J12: Conn_01x06_Socket, Connector_Molex:Molex_PicoBlade_53048-0610_1x06_P1.25mm_Horizontal, symbol Connector:Conn_01x06_Socket
- added R1, R2, R3, R4, R5: Resistor 82Ω, Resistor_THT:R_Axial_DIN0207_L6.3mm_D2.5mm_P7.62mm_Horizontal, symbol ScottoKeebs:Placeholder_Resistor
- added U2: Arduino_Pro_Micro, ScottoKeebs_MCU:Arduino_Pro_Micro, symbol ScottoKeebs:MCU_Arduino_Pro_Micro
Connections:
- net Caps Led: now also J10.3 (Pin_3)
- net LED PWR: now also U1.30 (5v), J10.6 (Pin_6); no longer TP4.1, U1.27 (3.3v)
- net Numpad Led: now also J10.2 (Pin_2)
- net at J7.5 (Pin_5), S12.1, S19.1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: now also S33.1
- net at D29.2 (A), D30.2 (A): now also D31.2 (A), D32.2 (A), D67.2 (A), J12.6 (Pin_6)
- net at D29.1 (K): now also R1.1
- net at D30.1 (K): now also R2.1
- net Power LED GND: now reaches U1.4 (GND)
- net Power LED GND: now also J10.1 (Pin_1)
- new net: J12.4 (Pin_4), R2.2
- new net: D67.1 (K), R5.1
- new net: D31.1 (K), R3.1
- new net: J12.3 (Pin_3), R3.2
- new net: J12.1 (Pin_1), R5.2
- new net: J12.2 (Pin_2), R4.2
- new net: J12.5 (Pin_5), R1.2
- new net: D32.1 (K), R4.1
- new net Battery LED: J10.5 (Pin_5), U2.20 (A3/PF4)
- new net Drive LED: J10.4 (Pin_4), U2.19 (A2/PF5)
- new net Trackpoint PWR: TP4.1, U1.27 (3.3v)
Other:
- note added: "Battery LED"
- note added: "Caps Lock"
- note added: "Drive Activity"
- note added: "Number Pad"
- note added: "Power"
- moved on the sheet: D29, D30, J11, J4, J8, TP1, TP10, TP2, TP3, TP4, TP5, TP6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

Commit message: added missing row and pullup resistors
Parts:
- removed J1, J2, J3, J8: Conn_01x05_Socket, Connector_Molex:Molex_PicoBlade_53048-0510_1x05_P1.25mm_Horizontal, symbol Connector:Conn_01x05_Socket
- added D29, D30, D31, D32, D40, D41, D42, D74, D75, D76, D78, D79, D80, D81: Diode, ScottoKeebs_Components:Diode_SOD-123, symbol ScottoKeebs:Placeholder_Diode
- added J13, J14, J15, J9: Conn_01x06_Socket, Connector_Molex:Molex_PicoBlade_53048-0610_1x06_P1.25mm_Horizontal, symbol Connector:Conn_01x06_Socket
- added R6, R7: Resistor 4.7k, ScottoKeebs_Components:Resistor_1206, symbol ScottoKeebs:Placeholder_Resistor
- added S29, S30, S31, S32, S40, S41, S42, S74, S75, S76, S77, S78, S79, S80: Keyswitch, ScottoKeebs_Choc:Choc_V1V2_1.00u, symbol ScottoKeebs:Placeholder_Keyswitch
- renumbered D36 to D43, D37 to D44, D38 to D45, D39 to D46, D40 to D47, D41 to D48, D42 to D49, D43 to D50, D44 to D51, D45 to D52, D46 to D53, D47 to D54, D48 to D55, D49 to D56, D50 to D57, D51 to D58, D52 to D59, D53 to D60, D54 to D61, D55 to D62, D56 to D63, D57 to D64, D58 to D65, D59 to D66, D60 to D67, D61 to D68, D62 to D69, D63 to D70, D64 to D71, D65 to D72, D66 to D73, D29 to D82, D30 to D83, D31 to D84, D32 to D85, D67 to D86, S36 to S43, S37 to S44, S38 to S45, S39 to S46, S40 to S47, S41 to S48, S42 to S49, S43 to S50, S44 to S51, S45 to S52, S46 to S53, S47 to S54, S48 to S55, S49 to S56, S50 to S57, S51 to S58, S52 to S59, S53 to S60, S54 to S61, S55 to S62, S56 to S63, S57 to S64, S58 to S65, S59 to S66, S60 to S67, S61 to S68, S62 to S69, S63 to S70, S64 to S71, S65 to S72, S66 to S73
Connections:
- net Caps Led: now also U1.14 (GP12); no longer U1.20 (GP23)
- net Col 0: now also U1.31 (GP11); no longer U1.2 (GP0)
- net Col 1: now also U1.21 (GP20); no longer U1.3 (GP1)
- net Col 10: now also U1.10 (GP6); no longer U1.16 (GP14)
- net Col 11: now also U1.11 (GP7); no longer U1.17 (GP15)
- net Col 12: now also U1.12 (GP8); no longer U1.18 (GP16)
- net Col 13: now also U1.13 (GP9); no longer U1.26 (GP29)
- net Col 2: now also U1.22 (GP22); no longer U1.6 (GP2)
- net Col 3: now also U1.23 (GP26); no longer U1.7 (GP3)
- net Col 4: now also U1.24 (GP27); no longer U1.10 (GP6)
- net Col 5: now also U1.25 (GP28); no longer U1.11 (GP7)
- net Col 6: now also U1.26 (GP29); no longer U1.12 (GP8)
- net Col 7: now also U1.7 (GP3); no longer U1.13 (GP9)
- net Col 8: now also U1.8 (GP4); no longer U1.14 (GP12)
- net Col 9: now also U1.9 (GP5); no longer U1.15 (GP13)
- net LED PWR: now also U2.21 (VCC); no longer U1.30 (5v)
- net Numpad Led: now also U1.6 (GP2); no longer U1.19 (GP21)
- net Power LED GND: now also U1.5 (GND); no longer U1.4 (GND)
- net Row 0: now also U1.20 (GP23), J9.6 (Pin_6); no longer U1.25 (GP28)
- net Row 1: now also U1.19 (GP21), J9.5 (Pin_5); no longer U1.24 (GP27)
- net Row 2: now also U1.18 (GP16), J9.4 (Pin_4); no longer U1.23 (GP26)
- net Row 3: now also U1.17 (GP15), J9.3 (Pin_3); no longer U1.22 (GP22)
- net Row 4: now also U1.16 (GP14), J9.2 (Pin_2); no longer U1.21 (GP20)
- net Trackpoint Clock: now also U1.3 (GP1), R7.1; no longer U1.9 (GP5)
- net Trackpoint Data: now also U1.2 (GP0), R6.1; no longer U1.8 (GP4)
- net Trackpoint GND: now also U1.4 (GND); no longer U1.29 (GND)
- net Trackpoint PWR: now also R6.2, R7.2
- net at J5.6 (Pin_6), S48.1, S55.1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: now also S76.1
- net at J5.5 (Pin_5), S47.1, S54.1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: now also S75.1
- net at J7.7 (Pin_7), S14.1, S21.1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: now also S42.1
- net at J5.7 (Pin_7), S49.1, S56.1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: now also S77.1
- net at J5.2 (Pin_2), S44.1, S51.1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: now also S79.1
- net at D15.1 (K), D16.1 (K), D17.1 (K)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: now also J13.4 (Pin_4), J14.3 (Pin_3)
- net at J5.4 (Pin_4), S46.1, S53.1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: now also S74.1
- net at J7.1 (Pin_1), S1.1, S15.1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: now also S29.1
- net at J5.1 (Pin_1), S43.1, S50.1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: now also S78.1
- net at J7.3 (Pin_3), S10.1, S17.1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: now also S31.1
- net at D64.1 (K), D65.1 (K), D66.1 (K)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: now also J15.4 (Pin_4)
- net at J7.6 (Pin_6), S13.1, S20.1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: now also S41.1
- net at D57.1 (K), D58.1 (K), D59.1 (K)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: now also J15.3 (Pin_3)
- net at D1.1 (K), D2.1 (K), D3.1 (K)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: now also J13.6 (Pin_6), J14.1 (Pin_1)
- net at D22.1 (K), D23.1 (K), D24.1 (K)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: now also J13.3 (Pin_3), J14.4 (Pin_4)
- net at J7.5 (Pin_5), S12.1, S19.1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: now also S40.1
- net at J7.4 (Pin_4), S11.1, S18.1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: now also S32.1
- net at D43.1 (K), D44.1 (K), D45.1 (K)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: now also J15.1 (Pin_1)
- net at D10.1 (K), D11.1 (K), D12.1 (K)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: now also J13.5 (Pin_5), J14.2 (Pin_2)
- net at D50.1 (K), D51.1 (K), D52.1 (K)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: now also J15.2 (Pin_2)
- net at D71.1 (K), D72.1 (K), D73.1 (K): now also D74.1 (K), D75.1 (K), D76.1 (K), D78.1 (K), J15.5 (Pin_5)
- net at J7.2 (Pin_2), S16.1, S2.1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: now also S30.1
- net at D33.1 (K), D34.1 (K), D35.1 (K): now also D29.1 (K), D30.1 (K), D31.1 (K), D32.1 (K), J13.2 (Pin_2), J14.5 (Pin_5)
- net at J5.3 (Pin_3), S45.1, S52.1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: now also S80.1
- new net: D76.2 (A), S76.2
- new net: D31.2 (A), S31.2
- new net: D79.1 (K), D80.1 (K), D81.1 (K), J15.6 (Pin_6)
- new net: D79.2 (A), S78.2
- new net: D80.2 (A), S79.2
- new net: D40.1 (K), D41.1 (K), D42.1 (K), J13.1 (Pin_1), J14.6 (Pin_6)
- new net: D41.2 (A), S41.2
- new net: D29.2 (A), S29.2
- new net: D78.2 (A), S77.2
- new net: D40.2 (A), S40.2
- new net: D30.2 (A), S30.2
- new net: D81.2 (A), S80.2
- new net: D32.2 (A), S32.2
- new net: D75.2 (A), S75.2
- new net: D42.2 (A), S42.2
- new net: D74.2 (A), S74.2
- new net Row 5: J9.1 (Pin_1), U1.15 (GP13)
Other:
- moved on the sheet: J11, TP1, TP10, TP2, TP3, TP4, TP5, TP6, TP7, TP8, TP9, U1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
